File: PMOS_Transistors.sch (KiCad schematic (older format))
At the start: 2 parts

Commit message: Updated component library
Parts:
- removed U? (x2): SI4463CDY, symbol SI4463CDY
- added Q? (x2): SI4463CDY, ~, symbol SI4463CDY
Connections:
- wire segments 9 -> 10
Changed lines of the file:
@@
 EESchema Schematic File Version 2
-LIBS:power
-LIBS:device
-LIBS:transistors
-LIBS:conn
-LIBS:linear
-LIBS:regul
-LIBS:74xx
-LIBS:cmos4000
-LIBS:adc-dac
-LIBS:memory
-LIBS:xilinx
-LIBS:special
-LIBS:microcontrollers
-LIBS:dsp
-LIBS:microchip
-LIBS:analog_switches
-LIBS:motorola
-LIBS:texas
-LIBS:intel
-LIBS:audio
-LIBS:interface
-LIBS:digital-audio
-LIBS:philips
-LIBS:display
-LIBS:cypress
-LIBS:siliconi
-LIBS:opto
-LIBS:atmel
-LIBS:contrib
-LIBS:valves
-LIBS:power_supply-cache
+LIBS:power_supply
 EELAYER 27 0
 EELAYER END
 $Descr A4 11693 8268
 encoding utf-8
-Sheet 4 4
+Sheet 3 4
 Title ""
 Date "15 jun 2014"
@@
 Comment4 ""
 $EndDescr
-$Comp
-L SI4463CDY U?
-U 1 1 539DACDB
-P 5600 2200
-F 0 "U?" H 5600 1950 60  0000 C CNN
-F 1 "SI4463CDY" H 5600 2450 60  0000 C CNN
-F 2 "" H 5600 2150 60  0000 C CNN
-F 3 "" H 5600 2150 60  0000 C CNN
-	1    5600 2200
-	1    0    0    -1
-$EndComp
-$Comp
-L SI4463CDY U?
-U 1 1 539DACEA
-P 5600 2900
-F 0 "U?" H 5600 2650 60  0000 C CNN
-F 1 "SI4463CDY" H 5600 3150 60  0000 C CNN
-F 2 "" H 5600 2850 60  0000 C CNN
-F 3 "" H 5600 2850 60  0000 C CNN
-	1    5600 2900
-	1    0    0    -1
-$EndComp
 Text HLabel 4850 2050 0    60   BiDi ~ 0
 S
-Text HLabel 4850 2350 0    60   BiDi ~ 0
+Text HLabel 4850 2250 0    60   BiDi ~ 0
 G
 Text HLabel 6250 2050 2    60   BiDi ~ 0
 D
+Connection ~ 5050 2250
 Wire Wire Line
-	5150 3050 5050 3050
+	4850 2050 5650 2050
+Connection ~ 4950 2050
+$Comp
+L SI4463CDY Q?
+U 1 1 539E1AB4
+P 5650 2300
+F 0 "Q?" H 5800 2400 60  0000 C CNN
+F 1 "SI4463CDY" H 5650 2550 60  0000 C CNN
+F 2 "~" H 5650 2250 60  0000 C CNN
+F 3 "~" H 5650 2250 60  0000 C CNN
+	1    5650 2300
+	0    -1   -1   0
+$EndComp
+$Comp
+L SI4463CDY Q?
+U 1 1 539E1ACB
+P 5650 2900
+F 0 "Q?" H 5800 3000 60  0000 C CNN
+F 1 "SI4463CDY" H 5650 3150 60  0000 C CNN
+F 2 "~" H 5650 2850 60  0000 C CNN
+F 3 "~" H 5650 2850 60  0000 C CNN
+	1    5650 2900
+	0    -1   -1   0
+$EndComp
 Wire Wire Line
-	5050 3050 5050 2350
+	4950 2650 5650 2650
 Wire Wire Line
-	4850 2350 5150 2350
-Connection ~ 5050 2350
+	4950 2650 4950 2050
 Wire Wire Line
-	5150 2750 4950 2750
+	5650 2550 6150 2550
 Wire Wire Line
-	4950 2750 4950 2050
+	6150 2050 6150 3150
 Wire Wire Line
-	4850 2050 5150 2050
-Connection ~ 4950 2050
+	6150 2050 6250 2050
 Wire Wire Line
-	6050 2050 6250 2050
+	6150 3150 5650 3150
+Connection ~ 6150 2550
 Wire Wire Line
-	6150 2050 6150 2750
+	5050 2850 5450 2850
 Wire Wire Line
-	6150 2750 6050 2750
-Connection ~ 6150 2050
+	5050 2250 5050 2850
+Wire Wire Line
+	4850 2250 5450 2250
 $EndSCHEMATC
